File: LightControllerBasic.kicad_pcb (KiCad board)
At the start: 2 copper layers, 140 x 50 mm, 71 parts, among them J1 Conn_01x08_Female, J2 Conn_01x08_Female, J3 Conn_01x08_Female, J4 Conn_01x08_Female, J5 Conn_01x08_Female, J6 Conn_01x08_Female, J7 Conn_01x08_Female, J8 Conn_01x08_Female, J9 Conn_01x02_Female, K1 HONGFA-HFD3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

Commit message: minor adjustments
Parts:
- removed the kibuzzard-62501B9E at (180.9, 93.5)
- removed kibuzzard-62501BA5: G***, kibuzzard-62501BA5
- added D17: LED, LED_SMD:LED_0603_1608Metric, B.Cu at (175.0, 90.0)
- added D18: LED, LED_SMD:LED_0603_1608Metric, B.Cu at (175.0, 88.0)
- added D19: D_Schottky, Diode_SMD:D_SMA, B.Cu at (167.5, 93.5)
- added R17: 2k2, Resistor_SMD:R_0603_1608Metric, B.Cu at (171.0, 90.0)
- added R18: 680, Resistor_SMD:R_0603_1608Metric, B.Cu at (171.0, 88.0)
- added kibuzzard-62551477: G***, kibuzzard-62551477, B.Cu at (180.5, 90.0)
- added kibuzzard-62551484: G***, kibuzzard-62551484, B.Cu at (180.5, 88.0)
- added kibuzzard-6255152E: G***, kibuzzard-6255152E, B.Cu at (182.0, 93.8)
- added kibuzzard-62551550: G***, kibuzzard-62551550, B.Cu at (182.0, 97.0)
- D1, D11, D13, D15, D3, D5, D7, D9: footprint Diode_SMD:D_SOD-323 -> Diode_SMD:D_SOD-323F
- H1, H2, H3, H4: footprint MountingHole:MountingHole_3.2mm_M3_ISO7380_Pad_TopBottom -> MountingHole:MountingHole_3.2mm_M3_DIN965_Pad_TopBottom
- U1: moved to F.Cu
- moved U1 4.75 mm to (171.0, 71.8)
- moved J9 2.50 mm to (175.0, 95.2)
Connections:
- J9 pad 1: +12V -> Net-(D19-A)
Routing:
- net +12V: track 95.5 -> 212.2 mm
- net OUT3: track 81.4 -> 108.3 mm, vias 1 -> 3
- net +5V: track 14.6 -> 36.3 mm, vias 0 -> 2
- net OUT1: track 105.0 -> 120.4 mm, vias 1 -> 3
- net OUT2: track 90.9 -> 106.3 mm, vias 0 -> 3
- net OUT6: track 29.4 -> 43.9 mm
- net OUT7: track 69.3 -> 80.7 mm, vias 1 -> 3
- net Net-(D19-A): track 0.00 -> 10.8 mm
- net OUT4: track 53.5 -> 61.2 mm, vias 1 -> 0
- net OUT0: track 115.3 -> 121.2 mm, vias 1 -> 3
- net OUT5: track 92.2 -> 96.8 mm, vias 1 -> 3
- net Net-(D18-K): track 0.00 -> 2.39 mm
- net Net-(D17-K): track 0.00 -> 2.39 mm
- net GND: vias 8 -> 10
- removed copper zone on F.Cu, net +12V
Other:
- board text added: "JLCJLCJLCJLC"
