File: LightControllerBasic.kicad_sch (KiCad schematic)
At the start: 63 parts, among them J1 Conn_01x08_Female, J2 Conn_01x08_Female, J3 Conn_01x08_Female, J4 Conn_01x08_Female, J5 Conn_01x08_Female, J6 Conn_01x08_Female, J7 Conn_01x08_Female, J8 Conn_01x08_Female, K1 HONGFA-HFD3, K2 HONGFA-HFD3, K3 HONGFA-HFD3, K4 HONGFA-HFD3, K5 HONGFA-HFD3, K6 HONGFA-HFD3, K7 HONGFA-HFD3, K8 HONGFA-HFD3, Q1 AO3400A, Q2 AO3400A, Q3 AO3400A, Q4 AO3400A, Q5 AO3400A, Q6 AO3400A, Q7 AO3400A, Q8 AO3400A

Commit message: minor adjustments
Parts:
- added D: D_Schottky, symbol Device:D_Schottky
- added U (x2): (no value), symbol Device:R_Small
- added U (x2): (no value), symbol Device:LED
- U: renamed from J1; value Conn_01x08_Female -> (none); footprint bouni:SPTAF_1_8_3_5_EL -> (none); now left out of the parts list
- U: renamed from J4; value Conn_01x08_Female -> (none); footprint bouni:SPTAF_1_8_3_5_EL -> (none); now left out of the parts list
- U: renamed from D12; value LED -> (none); footprint LED_SMD:LED_0603_1608Metric -> (none); LCSC (none) -> C72041
- U: renamed from R6; value 2k2 -> (none); footprint Resistor_SMD:R_0603_1608Metric -> (none); LCSC (none) -> C4190
- U: renamed from U1; now left out of the parts list
- U: renamed from D15; value 1N4148WS -> (none); footprint Diode_SMD:D_SOD-323 -> (none); LCSC (none) -> C2128
- U: renamed from R16; value 2k2 -> (none); footprint Resistor_SMD:R_0603_1608Metric -> (none); LCSC (none) -> C4190
- U: renamed from Q8; value AO3400A -> (none); footprint Package_TO_SOT_SMD:SOT-23 -> (none); LCSC (none) -> C344010
- U: renamed from R1; value 10k -> (none); footprint Resistor_SMD:R_0603_1608Metric -> (none); LCSC (none) -> C25804
- U: renamed from Q7; value AO3400A -> (none); footprint Package_TO_SOT_SMD:SOT-23 -> (none); LCSC (none) -> C344010
- U: renamed from Q1; value AO3400A -> (none); footprint Package_TO_SOT_SMD:SOT-23 -> (none); LCSC (none) -> C344010
- U: renamed from Q2; value AO3400A -> (none); footprint Package_TO_SOT_SMD:SOT-23 -> (none); LCSC (none) -> C344010
- U: renamed from R4; value 2k2 -> (none); footprint Resistor_SMD:R_0603_1608Metric -> (none); LCSC (none) -> C4190
- U: renamed from K3; value HONGFA-HFD3 -> (none); footprint bouni:HONGFA-HFD3 -> (none); now left out of the parts list
- U: renamed from J5; value Conn_01x08_Female -> (none); footprint bouni:SPTAF_1_8_3_5_EL -> (none); now left out of the parts list
- U: renamed from J2; value Conn_01x08_Female -> (none); footprint bouni:SPTAF_1_8_3_5_EL -> (none); now left out of the parts list
- U: renamed from J8; value Conn_01x08_Female -> (none); footprint bouni:SPTAF_1_8_3_5_EL -> (none); now left out of the parts list
- U: renamed from R8; value 2k2 -> (none); footprint Resistor_SMD:R_0603_1608Metric -> (none); LCSC (none) -> C4190
- U: renamed from D10; value LED -> (none); footprint LED_SMD:LED_0603_1608Metric -> (none); LCSC (none) -> C72041
- U: renamed from Q5; value AO3400A -> (none); footprint Package_TO_SOT_SMD:SOT-23 -> (none); LCSC (none) -> C344010
- U: renamed from H4; value MountingHole -> (none); footprint MountingHole:MountingHole_3.2mm_M3_ISO7380_Pad_TopBottom -> (none); now left out of the parts list
- U: renamed from R9; value 10k -> (none); footprint Resistor_SMD:R_0603_1608Metric -> (none); LCSC (none) -> C25804
- U: renamed from Q3; value AO3400A -> (none); footprint Package_TO_SOT_SMD:SOT-23 -> (none); LCSC (none) -> C344010
- U: renamed from K2; value HONGFA-HFD3 -> (none); footprint bouni:HONGFA-HFD3 -> (none); now left out of the parts list
- U: renamed from J3; value Conn_01x08_Female -> (none); footprint bouni:SPTAF_1_8_3_5_EL -> (none); now left out of the parts list
- U: renamed from D16; value LED -> (none); footprint LED_SMD:LED_0603_1608Metric -> (none); LCSC (none) -> C72041
- U: renamed from D6; value LED -> (none); footprint LED_SMD:LED_0603_1608Metric -> (none); LCSC (none) -> C72041
- U: renamed from R2; value 2k2 -> (none); footprint Resistor_SMD:R_0603_1608Metric -> (none); LCSC (none) -> C4190
- U: renamed from R7; value 10k -> (none); footprint Resistor_SMD:R_0603_1608Metric -> (none); LCSC (none) -> C25804
- U: renamed from Q4; value AO3400A -> (none); footprint Package_TO_SOT_SMD:SOT-23 -> (none); LCSC (none) -> C344010
- U: renamed from R10; value 2k2 -> (none); footprint Resistor_SMD:R_0603_1608Metric -> (none); LCSC (none) -> C4190
- U: renamed from H3; value MountingHole -> (none); footprint MountingHole:MountingHole_3.2mm_M3_ISO7380_Pad_TopBottom -> (none); now left out of the parts list
- U: renamed from R14; value 2k2 -> (none); footprint Resistor_SMD:R_0603_1608Metric -> (none); LCSC (none) -> C4190
- U: renamed from K4; value HONGFA-HFD3 -> (none); footprint bouni:HONGFA-HFD3 -> (none); now left out of the parts list
- U: renamed from R5; value 10k -> (none); footprint Resistor_SMD:R_0603_1608Metric -> (none); LCSC (none) -> C25804
- U: renamed from J6; value Conn_01x08_Female -> (none); footprint bouni:SPTAF_1_8_3_5_EL -> (none); now left out of the parts list
- U: renamed from D1; value 1N4148WS -> (none); footprint Diode_SMD:D_SOD-323 -> (none); LCSC (none) -> C2128
- U: renamed from R12; value 2k2 -> (none); footprint Resistor_SMD:R_0603_1608Metric -> (none); LCSC (none) -> C4190
- U: renamed from R11; value 10k -> (none); footprint Resistor_SMD:R_0603_1608Metric -> (none); LCSC (none) -> C25804
- U: renamed from U2; now left out of the parts list
- U: renamed from R13; value 10k -> (none); footprint Resistor_SMD:R_0603_1608Metric -> (none); LCSC (none) -> C25804
- U: renamed from D8; value LED -> (none); footprint LED_SMD:LED_0603_1608Metric -> (none); LCSC (none) -> C72041
- U: renamed from D2; value LED -> (none); footprint LED_SMD:LED_0603_1608Metric -> (none); LCSC (none) -> C72041
- U: renamed from D7; value 1N4148WS -> (none); footprint Diode_SMD:D_SOD-323 -> (none); LCSC (none) -> C2128
- U: renamed from Q6; value AO3400A -> (none); footprint Package_TO_SOT_SMD:SOT-23 -> (none); LCSC (none) -> C344010
- U: renamed from R3; value 10k -> (none); footprint Resistor_SMD:R_0603_1608Metric -> (none); LCSC (none) -> C25804
- U: renamed from K8; value HONGFA-HFD3 -> (none); footprint bouni:HONGFA-HFD3 -> (none); now left out of the parts list
- U: renamed from D13; value 1N4148WS -> (none); footprint Diode_SMD:D_SOD-323 -> (none); LCSC (none) -> C2128
- U: renamed from D11; value 1N4148WS -> (none); footprint Diode_SMD:D_SOD-323 -> (none); LCSC (none) -> C2128
- U: renamed from H1; value MountingHole -> (none); footprint MountingHole:MountingHole_3.2mm_M3_ISO7380_Pad_TopBottom -> (none); now left out of the parts list
- U: renamed from J7; value Conn_01x08_Female -> (none); footprint bouni:SPTAF_1_8_3_5_EL -> (none); now left out of the parts list
- U: renamed from D4; value LED -> (none); footprint LED_SMD:LED_0603_1608Metric -> (none); LCSC (none) -> C72041
- U: renamed from D3; value 1N4148WS -> (none); footprint Diode_SMD:D_SOD-323 -> (none); LCSC (none) -> C2128
- U: renamed from K6; value HONGFA-HFD3 -> (none); footprint bouni:HONGFA-HFD3 -> (none); now left out of the parts list
- U: renamed from D14; value LED -> (none); footprint LED_SMD:LED_0603_1608Metric -> (none); LCSC (none) -> C72041
- U: renamed from R15; value 10k -> (none); footprint Resistor_SMD:R_0603_1608Metric -> (none); LCSC (none) -> C25804
- U: renamed from K7; value HONGFA-HFD3 -> (none); footprint bouni:HONGFA-HFD3 -> (none); now left out of the parts list
- U: renamed from D5; value 1N4148WS -> (none); footprint Diode_SMD:D_SOD-323 -> (none); LCSC (none) -> C2128
- U: renamed from D9; value 1N4148WS -> (none); footprint Diode_SMD:D_SOD-323 -> (none); LCSC (none) -> C2128
- U: renamed from K1; value HONGFA-HFD3 -> (none); footprint bouni:HONGFA-HFD3 -> (none); now left out of the parts list
- U: renamed from K5; value HONGFA-HFD3 -> (none); footprint bouni:HONGFA-HFD3 -> (none); now left out of the parts list
- U: renamed from H2; value MountingHole -> (none); footprint MountingHole:MountingHole_3.2mm_M3_ISO7380_Pad_TopBottom -> (none); now left out of the parts list
- renumbered J9 to U
Connections:
- net +12V: now also D.1 (K), U.2 (A); no longer U.1 (Pin_1)
- net +5V: now also U.2 (A)
- net GND: now also U.2, U.2
- new net: U.1, U.1 (K) (x2)
- new net: D.2 (A), U.1 (Pin_1)
